File: eagle/pool-chemistry-v2.brd (EAGLE design)
At the start: 38.7 x 31.8 mm, 24 parts, among them IC1 MCP1703CB, P10 10k, P15 15k

Commit message: power and LDO labeling
Parts:
- BAT: value 5v -> (none)
- renumbered IC1 to LDO
Connections:
- net TOUCH1: now also ESPWROOM.12, PAD1.1; no longer ESPWROOM.25, PAD2.1
- net TOUCH2: now also ESPWROOM.25, PAD2.1; no longer ESPWROOM.12, PAD1.1
Routing:
- net TOUCH2: track 4.59 -> 17.1 mm
- net TOUCH1: track 17.1 -> 4.59 mm
Changed lines of the file:
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@@
 <text x="10.16" y="25.4" size="1.778" layer="25">+</text>
 <text x="10.16" y="17.78" size="1.778" layer="25">+</text>
+<text x="42.545" y="16.51" size="1.778" layer="38" rot="MR0">+</text>
+<text x="42.545" y="13.97" size="1.778" layer="38" rot="MR0">-</text>
 </plain>
 <attributes>
@@
 <attribute name="VALUE" x="30.48" y="26.035" size="1.27" layer="28" rot="MR0"/>
 </element>
-<element name="IC1" library="linear" library_urn="urn:adsk.eagle:library:262" package="SOT23" package3d_urn="urn:adsk.eagle:package:16489/2" value="MCP1703CB" x="26.035" y="12.065" smashed="yes" rot="MR0">
+<element name="LDO" library="linear" library_urn="urn:adsk.eagle:library:262" package="SOT23" package3d_urn="urn:adsk.eagle:package:16489/2" value="MCP1703CB" x="26.035" y="12.065" smashed="yes" rot="MR0">
 <attribute name="NAME" x="27.94" y="13.97" size="1.27" layer="26" rot="MR0"/>
 <attribute name="POPULARITY" value="19" x="26.035" y="12.065" size="1.778" layer="28" rot="MR0" display="off"/>
 <attribute name="VALUE" x="27.94" y="8.89" size="1.27" layer="28" rot="MR0"/>
 </element>
-<element name="BAT" library="pinhead" library_urn="urn:adsk.eagle:library:325" package="1X02" package3d_urn="urn:adsk.eagle:package:22435/2" value="5v" x="39.37" y="15.875" smashed="yes" rot="R90">
+<element name="BAT" library="pinhead" library_urn="urn:adsk.eagle:library:325" package="1X02" package3d_urn="urn:adsk.eagle:package:22435/2" value="" x="39.37" y="15.875" smashed="yes" rot="R90">
 <attribute name="NAME" x="37.5412" y="14.5288" size="1.27" layer="25" ratio="10" rot="R90"/>
 <attribute name="POPULARITY" value="98" x="39.37" y="15.875" size="1.778" layer="27" rot="R90" display="off"/>
-<attribute name="VALUE" x="42.545" y="13.335" size="1.27" layer="27" rot="R90"/>
+<attribute name="VALUE" x="43.18" y="15.24" size="1.27" layer="27" rot="R90"/>
 </element>
 <element name="PAD1" library="wirepad" library_urn="urn:adsk.eagle:library:412" package="SMD2,54-5,08" package3d_urn="urn:adsk.eagle:package:30841/1" value="" x="20.955" y="15.24" smashed="yes" rot="MR0">
@@
 <wire x1="30.48" y1="29.845" x2="30.61" y2="29.715" width="0.1524" layer="16"/>
 <wire x1="30.61" y1="29.715" x2="30.61" y2="28.575" width="0.1524" layer="16"/>
-<contactref element="IC1" pad="2"/>
+<contactref element="LDO" pad="2"/>
 <wire x1="23.11135" y1="7.6482" x2="23.4668" y2="8.00365" width="0.1524" layer="16"/>
 <wire x1="16.51" y1="7.62" x2="16.5382" y2="7.6482" width="0.1524" layer="16"/>
@@
 <via x="26.67" y="26.67" extent="1-16" drill="0.35"/>
 <wire x1="26.67" y1="29.29" x2="26.67" y2="26.67" width="0.1524" layer="1"/>
-<contactref element="IC1" pad="1"/>
+<contactref element="LDO" pad="1"/>
 <wire x1="27.305" y1="8.255" x2="26.985" y2="8.575" width="0.1524" layer="16"/>
 <wire x1="26.985" y1="8.575" x2="26.985" y2="10.965" width="0.1524" layer="16"/>
@@
 <wire x1="32.4" y1="10.005" x2="31.115" y2="11.29" width="0.1524" layer="1"/>
 </signal>
-<signal name="TOUCH1">
+<signal name="TOUCH2">
 <contactref element="ESPWROOM" pad="25"/>
 <wire x1="34.4" y1="12.78" x2="32.94" y2="12.78" width="0.1524" layer="1"/>
@@
 </signal>
 <signal name="VSS">
-<contactref element="IC1" pad="3"/>
+<contactref element="LDO" pad="3"/>
 <contactref element="BAT" pad="2"/>
 <wire x1="26.035" y1="13.165" x2="26.84" y2="13.97" width="0.1524" layer="16"/>
@@
 <wire x1="26.84" y1="13.97" x2="36.195" y2="13.97" width="0.1524" layer="16"/>
 </signal>
-<signal name="TOUCH2">
+<signal name="TOUCH1">
 <contactref element="ESPWROOM" pad="12"/>
 <contactref element="PAD1" pad="1"/>

Commit message: oshpark review changes for board - manufactured
Routing:
- net TEMPSIG: track 57.8 -> 56.7 mm
- net ORPDATA: track 31.3 -> 32.2 mm
Changed lines of the file:
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@@
 <text x="10.16" y="25.4" size="1.778" layer="25">+</text>
 <text x="10.16" y="17.78" size="1.778" layer="25">+</text>
-<text x="42.545" y="16.51" size="1.778" layer="38" rot="MR0">+</text>
-<text x="42.545" y="13.97" size="1.778" layer="38" rot="MR0">-</text>
+<text x="42.545" y="16.51" size="1.778" layer="26" rot="MR0">+</text>
+<text x="42.545" y="13.97" size="1.778" layer="26" rot="MR0">-</text>
 </plain>
 <attributes>
@@
 <wire x1="21.085" y1="8.255" x2="22.86" y2="8.255" width="0.1524" layer="1"/>
 <via x="22.86" y="8.255" extent="1-16" drill="0.35"/>
-<wire x1="22.86" y1="8.255" x2="22.86" y2="15.24" width="0.1524" layer="16"/>
-<via x="22.86" y="15.24" extent="1-16" drill="0.35"/>
-<wire x1="22.86" y1="15.24" x2="25.4" y2="17.78" width="0.1524" layer="1"/>
-<wire x1="29.845" y1="17.78" x2="25.4" y2="17.78" width="0.1524" layer="1"/>
+<wire x1="24.765" y1="11.43" x2="22.86" y2="9.525" width="0.1524" layer="16"/>
+<wire x1="22.86" y1="8.255" x2="22.86" y2="9.525" width="0.1524" layer="16"/>
+<wire x1="24.765" y1="15.24" x2="24.765" y2="11.43" width="0.1524" layer="16"/>
+<via x="24.765" y="15.24" extent="1-16" drill="0.35"/>
+<wire x1="24.765" y1="15.24" x2="27.305" y2="17.78" width="0.1524" layer="1"/>
+<wire x1="29.845" y1="17.78" x2="27.305" y2="17.78" width="0.1524" layer="1"/>
 <wire x1="29.845" y1="17.78" x2="32.385" y2="15.24" width="0.1524" layer="1"/>
 </signal>
@@
 <wire x1="8.89" y1="10.03" x2="8.89" y2="8.255" width="0.1524" layer="1"/>
 <wire x1="8.89" y1="8.255" x2="8.89" y2="5.845" width="0.1524" layer="1"/>
-<via x="14.605" y="21.59" extent="1-16" drill="0.35"/>
-<wire x1="14.605" y1="21.59" x2="14.605" y2="13.97" width="0.1524" layer="16"/>
+<via x="14.605" y="22.225" extent="1-16" drill="0.35"/>
+<wire x1="14.605" y1="22.225" x2="14.605" y2="13.97" width="0.1524" layer="16"/>
 <wire x1="14.605" y1="13.97" x2="6.985" y2="13.97" width="0.1524" layer="16"/>
 <via x="8.89" y="8.255" extent="1-16" drill="0.35"/>
 <wire x1="6.985" y1="8.255" x2="8.89" y2="8.255" width="0.1524" layer="16"/>
 <wire x1="6.985" y1="13.97" x2="6.985" y2="8.255" width="0.1524" layer="16"/>
-<wire x1="14.605" y1="21.59" x2="16.32" y2="21.59" width="0.1524" layer="1"/>
-<wire x1="16.32" y1="21.59" x2="16.4" y2="21.67" width="0.1524" layer="1"/>
+<wire x1="16.4" y1="21.67" x2="16.32" y2="21.59" width="0.1524" layer="1"/>
+<wire x1="16.32" y1="21.59" x2="15.24" y2="21.59" width="0.1524" layer="1"/>
+<wire x1="15.24" y1="21.59" x2="14.605" y2="22.225" width="0.1524" layer="1"/>
 <contactref element="C2" pad="2"/>
 <wire x1="8.89" y1="5.845" x2="8.89" y2="8.255" width="0.1524" layer="16"/>

Commit message: updates to design with fixes from first manufacturing run
Parts:
- added C5: 0.1, rcl:C1206
- added P1: 10k, rcl:M1206
- moved C3 1.27 mm to (22.9, 28.6)
- moved C4 1.27 mm to (30.5, 28.6)
- moved PAD2 1.27 mm to (21.0, 20.3)
- moved PAD1 0.63 mm to (21.0, 14.6)
Connections:
- new net ENABLE: C5.1, ESPWROOM.3, P1.1
- net GND: now also C5.2
- net VDD: now also P1.2; no longer AP3602A-ORP.4, AP3602A-PH.4
- net VSS: now also AP3602A-ORP.4, AP3602A-PH.4
Routing:
- net VSS: track 15.0 -> 37.2 mm
- net ENABLE: track 0.00 -> 15.6 mm, vias 0 -> 1
- net VDD: track 149.4 -> 139.3 mm
- net GND: track 165.7 -> 170.8 mm
- net ORP+5: track 29.5 -> 28.0 mm
- net TEMPSIG: track 56.7 -> 55.9 mm
- net TOUCH2: track 17.1 -> 16.6 mm
