File: eagle/pool-chemistry-v2.sch (EAGLE design)
At the start: 17 parts, among them U1 ESP-WROOM-32

Commit message: discrete components placed and routed
Parts:
- renumbered R1 to L1K, R2 to O10, R3 to O15, R4 to P15, R5 to P10, U1 to ESPWROOM
Connections:
- removed net TEMPEN: ESPWROOM.IO27, PU.1
- net TEMPSIG: now also PU.1; no longer PU.2
- net VDD: now also PU.2
Other:
- moved on the sheet: PU, TEMP, UART

Commit message: added missing labels to voltage divided signals
Connections:
- removed net N$2: ESPWROOM.IO35, O10.2, O15.1
- removed net N$4: ESPWROOM.IO33, P10.2, P15.1
- net ORPSIG: now also ESPWROOM.IO35, O10.2, O15.1
- net PHSIG: now also ESPWROOM.IO33, P10.2, P15.1
Changed lines of the file:
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@@
 <wire x1="27.94" y1="13.97" x2="27.94" y2="69.85" width="0.1524" layer="91"/>
+</segment>
+<segment>
+<pinref part="ESPWROOM" gate="G$1" pin="IO35"/>
+<wire x1="43.18" y1="80.01" x2="27.94" y2="80.01" width="0.1524" layer="91"/>
+<pinref part="O10" gate="G$1" pin="2"/>
+<pinref part="O15" gate="G$1" pin="1"/>
+<junction x="27.94" y="80.01"/>
+<label x="33.02" y="81.28" size="1.778" layer="95"/>
 </segment>
 </net>
@@
 <pinref part="P10" gate="G$1" pin="1"/>
 <wire x1="33.02" y1="64.77" x2="33.02" y2="-16.51" width="0.1524" layer="91"/>
+</segment>
+<segment>
+<pinref part="P10" gate="G$1" pin="2"/>
+<pinref part="P15" gate="G$1" pin="1"/>
+<pinref part="ESPWROOM" gate="G$1" pin="IO33"/>
+<wire x1="43.18" y1="74.93" x2="20.32" y2="74.93" width="0.1524" layer="91"/>
+<junction x="20.32" y="74.93"/>
+<label x="10.16" y="73.66" size="1.778" layer="95"/>
 </segment>
 </net>
@@
 </segment>
 </net>
-<net name="N$2" class="0">
-<segment>
-<pinref part="ESPWROOM" gate="G$1" pin="IO35"/>
-<wire x1="43.18" y1="80.01" x2="27.94" y2="80.01" width="0.1524" layer="91"/>
-<pinref part="O10" gate="G$1" pin="2"/>
-<pinref part="O15" gate="G$1" pin="1"/>
-<junction x="27.94" y="80.01"/>
-</segment>
-</net>
-<net name="N$4" class="0">
-<segment>
-<pinref part="P10" gate="G$1" pin="2"/>
-<pinref part="P15" gate="G$1" pin="1"/>
-<pinref part="ESPWROOM" gate="G$1" pin="IO33"/>
-<wire x1="43.18" y1="74.93" x2="20.32" y2="74.93" width="0.1524" layer="91"/>
-<junction x="20.32" y="74.93"/>
-</segment>
-</net>

Commit message: added ph, orp and esp ground caps
Parts:
- added C1, C2, C3: 0.1, rcl:C-USC1206
- added C4: 47, rcl:C-USC1206
Connections:
- new net ORPDATA: C2.2, ESPWROOM.IO35, O10.2, O15.1
- new net PHDATA: C1.2, ESPWROOM.IO33, P10.2, P15.1
- net GND: now also C1.1, C2.1, C3.2, C4.2
- net ORPSIG: no longer ESPWROOM.IO35, O10.2, O15.1
- net PHSIG: no longer ESPWROOM.IO33, P10.2, P15.1
- net VDD: now also C3.1, C4.1
Other:
- moved on the sheet: P10, P15

Commit message: added larger touch pads and LDO
Parts:
- removed TP1: TPTP20SQ, testpad:TPTP20SQ
- added BAT: 5v, pinhead:PINHD-1X2
- added IC1: MCP1703CB, linear:MCP1703CB
- added PAD1, PAD2: (no value), wirepad:SMD5
Connections:
- removed net TOUCH: ESPWROOM.IO0, TP1.TP
- new net TOUCH1: ESPWROOM.IO0, PAD2.P
- new net TOUCH2: ESPWROOM.IO27, PAD1.P
- new net VSS: BAT.2, IC1.VI
- net GND: now also BAT.1, IC1.GND
- net VDD: now also IC1.VO
Changed lines of the file:
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@@
 <setting verticaltext="up"/>
 </settings>
-<grid distance="50" unitdist="mil" unit="mil" style="lines" multiple="1" display="no" altdistance="0.01" altunitdist="inch" altunit="inch"/>
+<grid distance="0.1" unitdist="inch" unit="inch" style="lines" multiple="1" display="no" altdistance="0.01" altunitdist="inch" altunit="inch"/>
 <layers>
 <layer number="1" name="Top" color="4" fill="1" visible="no" active="no"/>
@@
 <part name="O10" library="rcl" library_urn="urn:adsk.eagle:library:334" deviceset="R-US_" device="M1206" package3d_urn="urn:adsk.eagle:package:23566/2" value="10k"/>
 <part name="O15" library="rcl" library_urn="urn:adsk.eagle:library:334" deviceset="R-US_" device="M1206" package3d_urn="urn:adsk.eagle:package:23566/2" value="15k"/>
-<part name="TP1" library="testpad" library_urn="urn:adsk.eagle:library:385" deviceset="TP" device="TP20SQ" package3d_urn="urn:adsk.eagle:package:27980/1"/>
 <part name="P15" library="rcl" library_urn="urn:adsk.eagle:library:334" deviceset="R-US_" device="M1206" package3d_urn="urn:adsk.eagle:package:23566/2" value="15k"/>
 <part name="P10" library="rcl" library_urn="urn:adsk.eagle:library:334" deviceset="R-US_" device="M1206" package3d_urn="urn:adsk.eagle:package:23566/2" value="10k"/>
@@
 <part name="C4" library="rcl" library_urn="urn:adsk.eagle:library:334" deviceset="C-US" device="C1206" package3d_urn="urn:adsk.eagle:package:23618/2" value="47"/>
 <part name="GND12" library="supply1" library_urn="urn:adsk.eagle:library:371" deviceset="GND" device=""/>
+<part name="IC1" library="linear" library_urn="urn:adsk.eagle:library:262" deviceset="MCP1703" device="CB" package3d_urn="urn:adsk.eagle:package:16489/2"/>
+<part name="SUPPLY1" library="supply2" library_urn="urn:adsk.eagle:library:372" deviceset="VSS" device=""/>
+<part name="BAT" library="pinhead" library_urn="urn:adsk.eagle:library:325" deviceset="PINHD-1X2" device="" package3d_urn="urn:adsk.eagle:package:22435/2" value="5v"/>
+<part name="PAD1" library="wirepad" library_urn="urn:adsk.eagle:library:412" deviceset="SMD5" device="" package3d_urn="urn:adsk.eagle:package:30841/1"/>
+<part name="PAD2" library="wirepad" library_urn="urn:adsk.eagle:library:412" deviceset="SMD5" device="" package3d_urn="urn:adsk.eagle:package:30841/1"/>
 </parts>
 <sheets>
@@
 <attribute name="VALUE" x="31.242" y="81.28" size="1.778" layer="96" rot="R90"/>
 </instance>
-<instance part="TP1" gate="G$1" x="104.14" y="57.15" smashed="yes" rot="R180">
-<attribute name="NAME" x="105.41" y="55.88" size="1.778" layer="95" rot="R270"/>
-<attribute name="TP_SIGNAL_NAME" x="102.87" y="58.42" size="1.778" layer="97" rot="R180"/>
-</instance>
 <instance part="P15" gate="G$1" x="10.16" y="80.01" smashed="yes" rot="R90">
 <attribute name="NAME" x="8.6614" y="76.2" size="1.778" layer="95" rot="R90"/>
@@
 <instance part="GND12" gate="1" x="-10.16" y="88.9" smashed="yes">
 <attribute name="VALUE" x="-12.7" y="86.36" size="1.778" layer="96"/>
+</instance>
+<instance part="IC1" gate="G$1" x="1.27" y="111.76" smashed="yes">
+<attribute name="NAME" x="-6.35" y="117.475" size="1.778" layer="95"/>
+<attribute name="VALUE" x="-6.35" y="114.935" size="1.778" layer="96"/>
+</instance>
+<instance part="SUPPLY1" gate="G$1" x="-15.24" y="106.68" smashed="yes">
+<attribute name="VALUE" x="-17.145" y="101.981" size="1.778" layer="96"/>
+</instance>
+<instance part="BAT" gate="G$1" x="-25.4" y="99.06" smashed="yes" rot="R180">
+<attribute name="NAME" x="-19.05" y="93.345" size="1.778" layer="95" rot="R180"/>
+<attribute name="VALUE" x="-19.05" y="104.14" size="1.778" layer="96" rot="R180"/>
+</instance>
+<instance part="PAD1" gate="1" x="45.72" y="24.13" smashed="yes" rot="R90">
+<attribute name="NAME" x="43.8658" y="22.987" size="1.778" layer="95" rot="R90"/>
+<attribute name="VALUE" x="49.022" y="22.987" size="1.778" layer="96" rot="R90"/>
+</instance>
+<instance part="PAD2" gate="1" x="101.6" y="54.61" smashed="yes" rot="R90">
+<attribute name="NAME" x="99.7458" y="53.467" size="1.778" layer="95" rot="R90"/>
+<attribute name="VALUE" x="104.902" y="53.467" size="1.778" layer="96" rot="R90"/>
 </instance>
 </instances>
@@
 <wire x1="35.56" y1="106.68" x2="35.56" y2="111.76" width="0.1524" layer="91"/>
 <junction x="35.56" y="111.76"/>
+<pinref part="IC1" gate="G$1" pin="VO"/>
+<wire x1="11.43" y1="111.76" x2="29.21" y2="111.76" width="0.1524" layer="91"/>
+<junction x="29.21" y="111.76"/>
 </segment>
 <segment>
@@
 <segment>
 <pinref part="GND12" gate="1" pin="GND"/>
-<wire x1="-10.16" y1="91.44" x2="10.16" y2="91.44" width="0.1524" layer="91"/>
+<wire x1="-10.16" y1="91.44" x2="1.27" y2="91.44" width="0.1524" layer="91"/>
 <pinref part="ESPWROOM" gate="G$1" pin="GND@1"/>
 <wire x1="38.1" y1="91.44" x2="38.1" y2="95.25" width="0.1524" layer="91"/>
@@
 <junction x="1.27" y="91.44"/>
 <junction x="10.16" y="91.44"/>
+<pinref part="IC1" gate="G$1" pin="GND"/>
+<wire x1="1.27" y1="104.14" x2="1.27" y2="96.52" width="0.1524" layer="91"/>
+<pinref part="BAT" gate="G$1" pin="1"/>
+<wire x1="1.27" y1="96.52" x2="1.27" y2="91.44" width="0.1524" layer="91"/>
+<wire x1="-22.86" y1="96.52" x2="1.27" y2="96.52" width="0.1524" layer="91"/>
+<junction x="1.27" y="96.52"/>
 </segment>
 </net>
@@
 </segment>
 </net>
-<net name="TOUCH" class="0">
+<net name="TOUCH1" class="0">
 <segment>
 <pinref part="ESPWROOM" gate="G$1" pin="IO0"/>
-<wire x1="91.44" y1="62.23" x2="104.14" y2="62.23" width="0.1524" layer="91"/>
+<wire x1="91.44" y1="62.23" x2="101.6" y2="62.23" width="0.1524" layer="91"/>
 <label x="96.52" y="62.23" size="1.778" layer="95"/>
-<pinref part="TP1" gate="G$1" pin="TP"/>
-<wire x1="104.14" y1="59.69" x2="104.14" y2="62.23" width="0.1524" layer="91"/>
+<pinref part="PAD2" gate="1" pin="P"/>
+<wire x1="101.6" y1="57.15" x2="101.6" y2="62.23" width="0.1524" layer="91"/>
 </segment>
 </net>
@@
 </segment>
 </net>
+<net name="VSS" class="0">
+<segment>
+<pinref part="IC1" gate="G$1" pin="VI"/>
+<wire x1="-8.89" y1="111.76" x2="-15.24" y2="111.76" width="0.1524" layer="91"/>
+<pinref part="SUPPLY1" gate="G$1" pin="VSS"/>
+<wire x1="-15.24" y1="109.22" x2="-15.24" y2="111.76" width="0.1524" layer="91"/>
+<pinref part="BAT" gate="G$1" pin="2"/>
+<wire x1="-22.86" y1="99.06" x2="-20.32" y2="99.06" width="0.1524" layer="91"/>
+<wire x1="-20.32" y1="99.06" x2="-20.32" y2="111.76" width="0.1524" layer="91"/>
+<wire x1="-20.32" y1="111.76" x2="-15.24" y2="111.76" width="0.1524" layer="91"/>
+<junction x="-15.24" y="111.76"/>
+</segment>
+</net>
+<net name="TOUCH2" class="0">
+<segment>
+<pinref part="ESPWROOM" gate="G$1" pin="IO27"/>
+<wire x1="43.18" y1="67.31" x2="39.37" y2="67.31" width="0.1524" layer="91"/>
+<wire x1="39.37" y1="67.31" x2="39.37" y2="31.75" width="0.1524" layer="91"/>
+<pinref part="PAD1" gate="1" pin="P"/>
+<wire x1="39.37" y1="31.75" x2="45.72" y2="31.75" width="0.1524" layer="91"/>
+<wire x1="45.72" y1="31.75" x2="45.72" y2="26.67" width="0.1524" layer="91"/>
+<label x="40.64" y="33.02" size="1.778" layer="95"/>
+</segment>
+</net>
